File: test1/test1.sch (KiCad schematic (older format))
At the start: 3 parts, among them J1 Conn_01x02_Male

Commit message: lection 3
Parts:
- D1: footprint (none) -> LED_SMD:LED_0805_2012Metric_Pad1.15x1.40mm_HandSolder
- J1: footprint (none) -> Connector_PinHeader_2.54mm:PinHeader_1x02_P2.54mm_Horizontal
- R1: footprint (none) -> Resistor_SMD:R_0805_2012Metric
Changed lines of the file:
@@
 F 0 "D1" V 6389 3982 50  0000 R CNN
 F 1 "LED" V 6298 3982 50  0000 R CNN
-F 2 "" H 6350 4100 50  0001 C CNN
+F 2 "LED_SMD:LED_0805_2012Metric_Pad1.15x1.40mm_HandSolder" H 6350 4100 50  0001 C CNN
 F 3 "~" H 6350 4100 50  0001 C CNN
 	1    6350 4100
@@
 F 0 "R1" H 6420 4746 50  0000 L CNN
 F 1 "510R" H 6420 4655 50  0000 L CNN
-F 2 "" V 6280 4700 50  0001 C CNN
+F 2 "Resistor_SMD:R_0805_2012Metric" V 6280 4700 50  0001 C CNN
 F 3 "~" H 6350 4700 50  0001 C CNN
 	1    6350 4700
@@
 F 0 "J1" H 7522 4324 50  0000 R CNN
 F 1 "Conn_01x02_Male" H 7522 4233 50  0000 R CNN
-F 2 "" H 7550 4350 50  0001 C CNN
+F 2 "Connector_PinHeader_2.54mm:PinHeader_1x02_P2.54mm_Horizontal" H 7550 4350 50  0001 C CNN
 F 3 "~" H 7550 4350 50  0001 C CNN
 	1    7550 4350
