File: InterfaceG850/InterfaceG850.kicad_pcb (KiCad board)
At the start: 2 copper layers, 27 parts, among them J1 USB_B_Micro, J2 Conn_01x11_Male, U1 FT232RL

Commit message: lecture commit
Parts:
- D1: value LED_Small -> PWR
- moved R11 47.2 mm to (117.0, 59.2), turned to 180 degrees
- moved F1 41.8 mm to (110.4, 64.1), turned to 180 degrees
- moved D1 39.0 mm to (112.5, 59.2), turned to 180 degrees
- moved C2 37.6 mm to (119.6, 65.2), turned to 270 degrees
- moved R4 37.0 mm to (141.0, 71.1), turned to 180 degrees
- moved C1 36.4 mm to (115.8, 65.2), turned to 270 degrees
- moved R5 33.9 mm to (116.6, 76.3), turned to 180 degrees
- moved J2 31.4 mm to (152.4, 63.5)
- moved R6 31.1 mm to (116.6, 74.1), turned to 180 degrees
- moved C3 28.9 mm to (123.3, 65.2), turned to 270 degrees
- moved JP1 27.7 mm to (115.9, 87.5)
- moved JP3 25.9 mm to (144.1, 66.0)
- moved R3 24.1 mm to (141.0, 83.8), turned to 180 degrees
- moved R1 23.8 mm to (141.0, 76.2), turned to 180 degrees
- moved R10 23.2 mm to (146.3, 71.1), turned to 180 degrees
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Connections:
- net Net-(F1-Pad2) renamed /VBUS
Routing:
- net +3V3: track 0.00 -> 17.3 mm
- net Net-(R4-Pad2): track 0.00 -> 17.3 mm
- net +5V: track 0.00 -> 16.5 mm
- net Net-(R3-Pad2): track 0.00 -> 15.6 mm
- net Net-(R2-Pad2): track 0.00 -> 13.9 mm, vias 0 -> 2
- net /VBUS: track 0.00 -> 12.6 mm
- net VCCIO: track 0.00 -> 10.3 mm
- net Net-(R1-Pad2): track 0.00 -> 9.07 mm
- net RXLED: track 0.00 -> 6.39 mm
- net TXLED: track 0.00 -> 6.18 mm
- net TXDCalc: track 0.00 -> 3.35 mm
- net RXDCalc: track 0.00 -> 3.35 mm
- net RTSCalc: track 0.00 -> 3.35 mm
- net CTSCalc: track 0.00 -> 3.08 mm
- net Net-(D3-Pad1): track 0.00 -> 3.05 mm
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Other:
- net class PWR added: clearance 0.2, trace_width 0.4, via_dia 0.8, via_drill 0.4

Commit message: 24.11.2020
Connections:
- net Net-(J1-Pad2) renamed /D-
- net Net-(J1-Pad3) renamed /D+
- net Net-(R5-Pad1) renamed /USBD_P
- net Net-(R6-Pad1) renamed /USBD_N
Routing:
- net +5V: track 16.5 -> 63.1 mm, vias 0 -> 2
- net VCCIO: track 10.3 -> 38.7 mm, vias 0 -> 2
- net /USBD_N: track 0.00 -> 10.8 mm
- net /USBD_P: track 0.00 -> 9.34 mm
- net /D+: track 0.00 -> 8.61 mm
- net RTSCalc: track 3.35 -> 11.7 mm
- net CTSCalc: track 3.08 -> 11.3 mm
- net TXDCalc: track 3.35 -> 11.3 mm
- net RXDCalc: track 3.35 -> 11.3 mm
- net /D-: track 0.00 -> 7.81 mm
- net VCCCalc: track 0.00 -> 7.62 mm
- net Net-(R4-Pad2): track 17.3 -> 16.1 mm
- added copper zone on B.Cu, net GND
- added copper zone on F.Cu, net GND
Other:
- board outline added: 50.4 x 37.1 mm
- board text added: "+3.3V"
- board text added: "+5V"
- board text added: "+PWR"
- board text added: "+RXD"
- board text added: "+TXD"
- board text added: "VCC Connect"
