File: InterfaceG850/InterfaceG850.kicad_pcb (KiCad board)
At the start: 2 copper layers, 50.4 x 37.1 mm, 27 parts, among them J1 USB_B_Micro, J2 Conn_01x11_Male, U1 FT232RL

Commit message: 27.11
Parts:
- added REF**: KiCad-Logo2_6mm_SilkScreen, hwreverse:KiCad-Logo2_6mm_SilkScreen, B.Cu at (143.3, 85.7)
Other:
- board text added: "Sharp G850 USB to Serial Converter"
- board text added: "ИУ10"

Commit message: Panda
Routing:
- net GND: vias 0 -> 91

Commit message: New OPLL Soundcard
Parts:
- added G***: LOGO, InterfaceG850:Panda_logo_slk, F.Cu at (109.9, 87.5)
