File: InterfaceG850/InterfaceG850.sch (KiCad schematic (older format))
At the start: 27 parts, among them J1 USB_B_Micro, J2 Conn_01x11_Male, U1 FT232RL

Commit message: C4
Parts:
- C4: value C_Small -> 0.1uF
Changed lines of the file:
@@
 P 4300 3700
 F 0 "C4" H 4392 3746 50  0000 L CNN
-F 1 "C_Small" H 4392 3655 50  0000 L CNN
+F 1 "0.1uF" H 4392 3655 50  0000 L CNN
 F 2 "" H 4300 3700 50  0001 C CNN
 F 3 "~" H 4300 3700 50  0001 C CNN

Commit message: Schema Ready
Parts:
- JP1: value SolderJumper_2_Open -> 3.3V VCCIO
- JP2: value SolderJumper_2_Open -> 5V VCCIO
- JP3: value SolderJumper_2_Open -> Calc Power from USB
Connections:
- net labels added: CTSCalc, RTSCalc, RXDCalc, RXLED, TXDCalc, TXLED, VCCCalc, VCCIO
- wire segments 74 -> 83
- no-connect marks 0 -> 15
Changed lines of the file:
@@
 encoding utf-8
 Sheet 1 1
-Title "USB to Serial Interface for SHarp PC-G850"
+Title "USB to Serial Interface for Sharp PC-G850"
 Date "2020-11-13"
 Rev ""
@@
 P 2150 4150
 F 0 "JP1" H 2150 4355 50  0000 C CNN
-F 1 "SolderJumper_2_Open" H 2150 4264 50  0000 C CNN
+F 1 "3.3V VCCIO" H 2150 4264 50  0000 C CNN
 F 2 "" H 2150 4150 50  0001 C CNN
 F 3 "~" H 2150 4150 50  0001 C CNN
@@
 P 3200 4150
 F 0 "JP2" H 3200 4355 50  0000 C CNN
-F 1 "SolderJumper_2_Open" H 3200 4264 50  0000 C CNN
+F 1 "5V VCCIO" H 3200 4264 50  0000 C CNN
 F 2 "" H 3200 4150 50  0001 C CNN
 F 3 "~" H 3200 4150 50  0001 C CNN
@@
 P 8150 4450
 F 0 "JP3" H 8150 4655 50  0000 C CNN
-F 1 "SolderJumper_2_Open" H 8150 4564 50  0000 C CNN
+F 1 "Calc Power from USB" H 8150 4564 50  0000 C CNN
 F 2 "" H 8150 4450 50  0001 C CNN
 F 3 "~" H 8150 4450 50  0001 C CNN
@@
 	1500 4150 1500 3800
 Wire Wire Line
-	2650 4150 2650 3800
+	2650 4150 2650 3900
 Connection ~ 2650 4150
 Wire Wire Line
@@
 	1    0    0    -1
 $EndComp
+Text GLabel 10100 2850 0    50   Output ~ 0
+RTSCalc
+Wire Wire Line
+	10100 2850 10300 2850
+Text GLabel 8700 2000 1    50   Input ~ 0
+RTSCalc
+Text GLabel 10100 3050 0    50   Input ~ 0
+RXDCalc
+Text GLabel 10100 3150 0    50   Output ~ 0
+TXDCalc
+Text GLabel 10100 3350 0    50   Input ~ 0
+CTSCalc
+Wire Wire Line
+	10100 3050 10300 3050
+Wire Wire Line
+	10100 3150 10300 3150
+Wire Wire Line
+	10100 3350 10300 3350
+Text GLabel 7500 2000 1    50   Output ~ 0
+RXDCalc
+Text GLabel 7900 2000 1    50   Input ~ 0
+TXDCalc
+Text GLabel 8300 2000 1    50   Output ~ 0
+CTSCalc
+Wire Wire Line
+	10300 2750 9550 2750
+Wire Wire Line
+	9550 2750 9550 2850
+Wire Wire Line
+	10300 2650 9900 2650
+Wire Wire Line
+	9900 2650 9900 2400
+$Comp
+L power:GND #PWR0101
+U 1 1 5FB4F765
+P 9550 2850
+F 0 "#PWR0101" H 9550 2600 50  0001 C CNN
+F 1 "GND" H 9555 2677 50  0000 C CNN
+F 2 "" H 9550 2850 50  0001 C CNN
+F 3 "" H 9550 2850 50  0001 C CNN
+	1    9550 2850
+	1    0    0    -1
+$EndComp
+Text GLabel 9900 2400 1    50   UnSpc ~ 0
+VCCCalc
+Text GLabel 8850 4450 2    50   UnSpc ~ 0
+VCCCalc
+Text GLabel 5900 1500 1    50   UnSpc ~ 0
+VCCIO
+Text GLabel 2650 3800 1    50   UnSpc ~ 0
+VCCIO
+Text GLabel 6800 3550 2    50   Output ~ 0
+RXLED
+Text GLabel 6800 3650 2    50   Output ~ 0
+TXLED
+Text GLabel 5550 5950 3    50   Output ~ 0
+RXLED
+Text GLabel 6550 5950 3    50   Output ~ 0
+TXLED
+Text GLabel 5550 5000 1    50   UnSpc ~ 0
+VCCIO
+Text GLabel 6550 5000 1    50   UnSpc ~ 0
+VCCIO
+NoConn ~ 10300 2550
+NoConn ~ 10300 2950
+NoConn ~ 10300 3450
+NoConn ~ 10300 3550
+NoConn ~ 6800 2950
+NoConn ~ 6800 3050
+NoConn ~ 6800 3150
+NoConn ~ 6800 3250
+NoConn ~ 6800 3750
+NoConn ~ 6800 3850
+NoConn ~ 6800 3950
+NoConn ~ 5200 3450
+NoConn ~ 5200 3650
+NoConn ~ 1450 3050
+$Comp
+L power:PWR_FLAG #FLG0101
+U 1 1 5FB6F554
+P 2650 3900
+F 0 "#FLG0101" H 2650 3975 50  0001 C CNN
+F 1 "PWR_FLAG" V 2650 4027 50  0001 L CNN
+F 2 "" H 2650 3900 50  0001 C CNN
+F 3 "~" H 2650 3900 50  0001 C CNN
+	1    2650 3900
+	0    -1   -1   0
+$EndComp
+Connection ~ 2650 3900
+Wire Wire Line
+	2650 3900 2650 3800
+$Comp
+L power:PWR_FLAG #FLG0102
+U 1 1 5FB7081C
+P 3950 1350
+F 0 "#FLG0102" H 3950 1425 50  0001 C CNN
+F 1 "PWR_FLAG" V 3950 1478 50  0001 L CNN
+F 2 "" H 3950 1350 50  0001 C CNN
+F 3 "~" H 3950 1350 50  0001 C CNN
+	1    3950 1350
+	0    1    1    0
+$EndComp
+NoConn ~ 10300 3250
 $EndSCHEMATC

Commit message: Added Footprints
Parts:
- C1, C2, C3, C4: footprint (none) -> Capacitor_SMD:C_0805_2012Metric_Pad1.18x1.45mm_HandSolder
- D1, D2, D3: footprint (none) -> LED_SMD:LED_0805_2012Metric_Pad1.15x1.40mm_HandSolder
- F1: footprint (none) -> Resistor_SMD:R_1210_3225Metric_Pad1.30x2.65mm_HandSolder
- J1: footprint (none) -> Connector_USB:USB_Micro-B_Molex-105017-0001
- J2: footprint (none) -> Connector_PinHeader_2.54mm:PinHeader_1x11_P2.54mm_Vertical
- JP1, JP2, JP3: footprint (none) -> Jumper:SolderJumper-2_P1.3mm_Open_RoundedPad1.0x1.5mm
- R1, R10, R11, R12, R13, R2, R3, R4, R5, R6, R7, R8, R9: footprint (none) -> Resistor_SMD:R_0805_2012Metric_Pad1.20x1.40mm_HandSolder
Changed lines of the file:
@@
 F 0 "J1" H 1207 3317 50  0000 C CNN
 F 1 "USB_B_Micro" H 1207 3226 50  0000 C CNN
-F 2 "" H 1300 2800 50  0001 C CNN
+F 2 "Connector_USB:USB_Micro-B_Molex-105017-0001" H 1300 2800 50  0001 C CNN
 F 3 "~" H 1300 2800 50  0001 C CNN
 	1    1150 2850
@@
 F 0 "J2" H 10472 3074 50  0000 R CNN
 F 1 "Conn_01x11_Male" H 10472 2983 50  0000 R CNN
-F 2 "" H 10500 3050 50  0001 C CNN
+F 2 "Connector_PinHeader_2.54mm:PinHeader_1x11_P2.54mm_Vertical" H 10500 3050 50  0001 C CNN
 F 3 "~" H 10500 3050 50  0001 C CNN
 	1    10500 3050
@@
 F 0 "R5" V 2404 2850 50  0000 C CNN
 F 1 "15R" V 2495 2850 50  0000 C CNN
-F 2 "" H 2600 2850 50  0001 C CNN
+F 2 "Resistor_SMD:R_0805_2012Metric_Pad1.20x1.40mm_HandSolder" H 2600 2850 50  0001 C CNN
 F 3 "~" H 2600 2850 50  0001 C CNN
 	1    2600 2850
@@
 F 0 "R6" V 2704 2950 50  0000 C CNN
 F 1 "15R" V 2795 2950 50  0000 C CNN
-F 2 "" H 2600 2950 50  0001 C CNN
+F 2 "Resistor_SMD:R_0805_2012Metric_Pad1.20x1.40mm_HandSolder" H 2600 2950 50  0001 C CNN
 F 3 "~" H 2600 2950 50  0001 C CNN
 	1    2600 2950
@@
 F 0 "C1" H 2842 1646 50  0000 L CNN
 F 1 "0.1uF" H 2842 1555 50  0000 L CNN
-F 2 "" H 2750 1600 50  0001 C CNN
+F 2 "Capacitor_SMD:C_0805_2012Metric_Pad1.18x1.45mm_HandSolder" H 2750 1600 50  0001 C CNN
 F 3 "~" H 2750 1600 50  0001 C CNN
 	1    2750 1600
@@
 F 0 "C2" H 3442 1646 50  0000 L CNN
 F 1 "10nF" H 3442 1555 50  0000 L CNN
-F 2 "" H 3350 1600 50  0001 C CNN
+F 2 "Capacitor_SMD:C_0805_2012Metric_Pad1.18x1.45mm_HandSolder" H 3350 1600 50  0001 C CNN
 F 3 "~" H 3350 1600 50  0001 C CNN
 	1    3350 1600
@@
 F 0 "C3" H 4042 1646 50  0000 L CNN
 F 1 "10uF" H 4042 1555 50  0000 L CNN
-F 2 "" H 3950 1600 50  0001 C CNN
+F 2 "Capacitor_SMD:C_0805_2012Metric_Pad1.18x1.45mm_HandSolder" H 3950 1600 50  0001 C CNN
 F 3 "~" H 3950 1600 50  0001 C CNN
 	1    3950 1600
@@
 F 0 "C4" H 4392 3746 50  0000 L CNN
 F 1 "0.1uF" H 4392 3655 50  0000 L CNN
-F 2 "" H 4300 3700 50  0001 C CNN
+F 2 "Capacitor_SMD:C_0805_2012Metric_Pad1.18x1.45mm_HandSolder" H 4300 3700 50  0001 C CNN
 F 3 "~" H 4300 3700 50  0001 C CNN
 	1    4300 3700
@@
 F 0 "R11" H 2541 5354 50  0000 R CNN
 F 1 "510R" H 2541 5445 50  0000 R CNN
-F 2 "" H 2600 5400 50  0001 C CNN
+F 2 "Resistor_SMD:R_0805_2012Metric_Pad1.20x1.40mm_HandSolder" H 2600 5400 50  0001 C CNN
 F 3 "~" H 2600 5400 50  0001 C CNN
 	1    2600 5400
@@
 F 0 "R12" H 5491 5604 50  0000 R CNN
 F 1 "510R" H 5491 5695 50  0000 R CNN
-F 2 "" H 5550 5650 50  0001 C CNN
+F 2 "Resistor_SMD:R_0805_2012Metric_Pad1.20x1.40mm_HandSolder" H 5550 5650 50  0001 C CNN
 F 3 "~" H 5550 5650 50  0001 C CNN
 	1    5550 5650
@@
 F 0 "R13" H 6491 5604 50  0000 R CNN
 F 1 "510R" H 6491 5695 50  0000 R CNN
-F 2 "" H 6550 5650 50  0001 C CNN
+F 2 "Resistor_SMD:R_0805_2012Metric_Pad1.20x1.40mm_HandSolder" H 6550 5650 50  0001 C CNN
 F 3 "~" H 6550 5650 50  0001 C CNN
 	1    6550 5650
@@
 F 0 "R1" V 7104 2550 50  0000 C CNN
 F 1 "100R" V 7195 2550 50  0000 C CNN
-F 2 "" H 7300 2550 50  0001 C CNN
+F 2 "Resistor_SMD:R_0805_2012Metric_Pad1.20x1.40mm_HandSolder" H 7300 2550 50  0001 C CNN
 F 3 "~" H 7300 2550 50  0001 C CNN
 	1    7300 2550
@@
 F 0 "R2" V 7504 2650 50  0000 C CNN
 F 1 "100R" V 7595 2650 50  0000 C CNN
-F 2 "" H 7700 2650 50  0001 C CNN
+F 2 "Resistor_SMD:R_0805_2012Metric_Pad1.20x1.40mm_HandSolder" H 7700 2650 50  0001 C CNN
 F 3 "~" H 7700 2650 50  0001 C CNN
 	1    7700 2650
@@
 F 0 "R3" V 7904 2750 50  0000 C CNN
 F 1 "100R" V 7995 2750 50  0000 C CNN
-F 2 "" H 8100 2750 50  0001 C CNN
+F 2 "Resistor_SMD:R_0805_2012Metric_Pad1.20x1.40mm_HandSolder" H 8100 2750 50  0001 C CNN
 F 3 "~" H 8100 2750 50  0001 C CNN
 	1    8100 2750
@@
 F 0 "R4" V 8304 2850 50  0000 C CNN
 F 1 "100R" V 8395 2850 50  0000 C CNN
-F 2 "" H 8500 2850 50  0001 C CNN
+F 2 "Resistor_SMD:R_0805_2012Metric_Pad1.20x1.40mm_HandSolder" H 8500 2850 50  0001 C CNN
 F 3 "~" H 8500 2850 50  0001 C CNN
 	1    8500 2850
@@
 F 0 "R7" H 7441 3154 50  0000 R CNN
 F 1 "10K" H 7441 3245 50  0000 R CNN
-F 2 "" H 7500 3200 50  0001 C CNN
+F 2 "Resistor_SMD:R_0805_2012Metric_Pad1.20x1.40mm_HandSolder" H 7500 3200 50  0001 C CNN
 F 3 "~" H 7500 3200 50  0001 C CNN
 	1    7500 3200
@@
 F 0 "R8" H 7841 3154 50  0000 R CNN
 F 1 "10K" H 7841 3245 50  0000 R CNN
-F 2 "" H 7900 3200 50  0001 C CNN
+F 2 "Resistor_SMD:R_0805_2012Metric_Pad1.20x1.40mm_HandSolder" H 7900 3200 50  0001 C CNN
 F 3 "~" H 7900 3200 50  0001 C CNN
 	1    7900 3200
@@
 F 0 "R9" H 8241 3154 50  0000 R CNN
 F 1 "10K" H 8241 3245 50  0000 R CNN
-F 2 "" H 8300 3200 50  0001 C CNN
+F 2 "Resistor_SMD:R_0805_2012Metric_Pad1.20x1.40mm_HandSolder" H 8300 3200 50  0001 C CNN
 F 3 "~" H 8300 3200 50  0001 C CNN
 	1    8300 3200
@@
 F 0 "R10" H 8641 3154 50  0000 R CNN
 F 1 "10K" H 8641 3245 50  0000 R CNN
-F 2 "" H 8700 3200 50  0001 C CNN
+F 2 "Resistor_SMD:R_0805_2012Metric_Pad1.20x1.40mm_HandSolder" H 8700 3200 50  0001 C CNN
 F 3 "~" H 8700 3200 50  0001 C CNN
 	1    8700 3200
@@
 F 0 "D1" V 2646 4980 50  0000 R CNN
 F 1 "LED_Small" V 2555 4980 50  0000 R CNN
-F 2 "" V 2600 5050 50  0001 C CNN
+F 2 "LED_SMD:LED_0805_2012Metric_Pad1.15x1.40mm_HandSolder" V 2600 5050 50  0001 C CNN
 F 3 "~" V 2600 5050 50  0001 C CNN
 	1    2600 5050
@@
 F 0 "D2" V 5596 5230 50  0000 R CNN
 F 1 "RX" V 5505 5230 50  0000 R CNN
-F 2 "" V 5550 5300 50  0001 C CNN
+F 2 "LED_SMD:LED_0805_2012Metric_Pad1.15x1.40mm_HandSolder" V 5550 5300 50  0001 C CNN
 F 3 "~" V 5550 5300 50  0001 C CNN
 	1    5550 5300
@@
 F 0 "D3" V 6596 5230 50  0000 R CNN
 F 1 "TX" V 6505 5230 50  0000 R CNN
-F 2 "" V 6550 5300 50  0001 C CNN
+F 2 "LED_SMD:LED_0805_2012Metric_Pad1.15x1.40mm_HandSolder" V 6550 5300 50  0001 C CNN
 F 3 "~" V 6550 5300 50  0001 C CNN
 	1    6550 5300
@@
 F 0 "F1" V 1825 1350 50  0000 C CNN
 F 1 "PTC 500mA" V 1916 1350 50  0000 C CNN
-F 2 "" H 2100 1150 50  0001 L CNN
+F 2 "Resistor_SMD:R_1210_3225Metric_Pad1.30x2.65mm_HandSolder" H 2100 1150 50  0001 L CNN
 F 3 "~" H 2050 1350 50  0001 C CNN
 	1    2050 1350
@@
 F 0 "JP1" H 2150 4355 50  0000 C CNN
 F 1 "3.3V VCCIO" H 2150 4264 50  0000 C CNN
-F 2 "" H 2150 4150 50  0001 C CNN
+F 2 "Jumper:SolderJumper-2_P1.3mm_Open_RoundedPad1.0x1.5mm" H 2150 4150 50  0001 C CNN
 F 3 "~" H 2150 4150 50  0001 C CNN
 	1    2150 4150
@@
 F 0 "JP2" H 3200 4355 50  0000 C CNN
 F 1 "5V VCCIO" H 3200 4264 50  0000 C CNN
-F 2 "" H 3200 4150 50  0001 C CNN
+F 2 "Jumper:SolderJumper-2_P1.3mm_Open_RoundedPad1.0x1.5mm" H 3200 4150 50  0001 C CNN
 F 3 "~" H 3200 4150 50  0001 C CNN
 	1    3200 4150
@@
 F 0 "JP3" H 8150 4655 50  0000 C CNN
 F 1 "Calc Power from USB" H 8150 4564 50  0000 C CNN
-F 2 "" H 8150 4450 50  0001 C CNN
+F 2 "Jumper:SolderJumper-2_P1.3mm_Open_RoundedPad1.0x1.5mm" H 8150 4450 50  0001 C CNN
 F 3 "~" H 8150 4450 50  0001 C CNN
 	1    8150 4450

Commit message: lecture commit
Parts:
- D1: value LED_Small -> PWR
Connections:
- net VBUS: now reaches F1.2, J1.1 (VBUS)
Changed lines of the file:
@@
 P 2600 5050
 F 0 "D1" V 2646 4980 50  0000 R CNN
-F 1 "LED_Small" V 2555 4980 50  0000 R CNN
+F 1 "PWR" V 2555 4980 50  0000 R CNN
 F 2 "LED_SMD:LED_0805_2012Metric_Pad1.15x1.40mm_HandSolder" V 2600 5050 50  0001 C CNN
 F 3 "~" V 2600 5050 50  0001 C CNN
@@
 Wire Wire Line
 	2600 5150 2600 5300
-Wire Wire Line
-	5550 5400 5550 5550
 Wire Wire Line
 	6550 5400 6550 5550
@@
 $EndComp
 NoConn ~ 10300 3250
+Text Label 1650 2150 1    50   ~ 0
+VBUS
+Wire Wire Line
+	5550 5400 5550 5550
 $EndSCHEMATC

Commit message: 24.11.2020
Connections:
- net USBD_P: now reaches R5.1, U1.15 (USBD+)
- net USBD_N: now reaches R6.1, U1.16 (USBD-)
- net D-: now reaches J1.2 (D-), R6.2
- net D+: now reaches J1.3 (D+), R5.2
Changed lines of the file:
@@
 Wire Wire Line
 	5550 5400 5550 5550
+Text Label 1700 2850 0    50   ~ 0
+D+
+Text Label 1700 2950 0    50   ~ 0
+D-
+Text Label 3650 2850 0    50   ~ 0
+USBD_P
+Text Label 3650 2950 0    50   ~ 0
+USBD_N
 $EndSCHEMATC
